Commit message: Reduce limits of the base joints in the URDF

File: share/urdf/pepper.urdf (robot description, URDF)
Before this commit: robot JulietteY20MP, 84 links, 83 joints
Joints:
- joint HipPitch: limit lower=-1.03847 upper=1.03847 effort=19.787 velocity=2.93276 -> lower=-0.346 upper=0.346 effort=19.787 velocity=2.93276
- joint HipRoll: limit lower=-0.514872 upper=0.514872 effort=10.1884 velocity=2.27032 -> lower=-0.257 upper=0.257 effort=10.1884 velocity=2.27032
- joint KneePitch: limit lower=-0.514872 upper=0.514872 effort=27.702 velocity=2.93276 -> lower=-0.1716 upper=0.1716 effort=27.702 velocity=2.93276

Commit message: New URDF

File: share/urdf/pepper.urdf (robot description, URDF)
Before this commit: robot JulietteY20MP, 84 links, 83 joints
Links:
- removed link ImuBaseGyrometer_frame
- removed link base_link
- added link Lgrasp_frame
- added link l_grasp_frame, mass 0
- added link r_grasp_frame, mass 0
- added link torso_base
Joints:
- removed joint GyrometerBase_sensor_fixedjoint
- removed joint base_link_fixedjoint
- added joint LGrasp: type fixed, parent l_wrist, child l_grasp_frame, origin xyz=0.05 0 0 rpy=-3.1415 0 1.5707, axis 1.0 0 0, limit lower=0.02 upper=0.98 effort=0.144 velocity=12.56
- added joint Lgrasp_frame_joint: type fixed, parent l_wrist, child Lgrasp_frame, origin xyz=0.070 0 0 rpy=3.1415 0 1.5707
- added joint RGrasp: type fixed, parent r_wrist, child r_grasp_frame, origin xyz=0.05 0 0 rpy=-3.1415 0 1.5707, axis 1.0 0 0, limit lower=0.02 upper=0.98 effort=0.144 velocity=12.56
- added joint torso_base_fixedjoint: type fixed, parent torso_base, child torso, origin xyz=-2e-05 0 0.139 rpy=0 0 0, axis 0 0 0
- joint AccelerometerBase_sensor_fixedjoint: origin xyz=0 0 -0.3 rpy=0 0 0 -> xyz=0.0147 -0.0017 -0.26319 rpy=0 0 0
- joint CameraBottom_sensor_fixedjoint: origin xyz=0.0936 0 0.0616 rpy=0 0.698132 0 -> xyz=0.09262 0 0.06177 rpy=0 0.698132 0
- joint CameraTop_sensor_fixedjoint: origin xyz=0.0868 0 0.1631 rpy=0 0 0 -> xyz=0.08601 0 0.16284 rpy=0 0 0
- joint HipPitch: child Pelvis -> Hip; limit lower=-0.346 upper=0.346 effort=19.787 velocity=2.93276 -> lower=-1.03847 upper=1.03847 effort=19.787 velocity=2.93276; origin xyz=0 0 -0.079 rpy=0 0 0 -> xyz=0 0 0.268 rpy=0 0 0; parent Hip -> Pelvis
- joint HipRoll: child Hip -> torso_base; limit lower=-0.257 upper=0.257 effort=10.1884 velocity=2.27032 -> lower=-0.514872 upper=0.514872 effort=10.1884 velocity=2.27032; origin xyz=2e-05 0 -0.139 rpy=0 0 0 -> xyz=0 0 0.079 rpy=0 0 0; parent torso -> Hip
- joint KneePitch: child Tibia -> Pelvis; limit lower=-0.1716 upper=0.1716 effort=27.702 velocity=2.93276 -> lower=-0.514872 upper=0.514872 effort=27.702 velocity=2.93276; origin xyz=0 0 -0.268 rpy=0 0 0 -> xyz=0 0 0 rpy=0 0 0; parent Pelvis -> Tibia
- joint LaserSensor/Front_sensor_fixedjoint: origin xyz=0.0562 0 -0.0692 rpy=0 0.349044 0 -> xyz=0.0562 0 -0.0692 rpy=0 0.349066 0
- joint LaserSensor/Left_sensor_fixedjoint: origin xyz=-0.018 0.0899 -0.0759 rpy=8.34035e-09 0.191982 1.5708 -> xyz=-0.018 0.0899 -0.0759 rpy=0 0.349066 1.5708
- joint LaserSensor/Right_sensor_fixedjoint: origin xyz=-0.018 -0.0899 -0.0759 rpy=4.08851e-07 0.191857 -1.60746 -> xyz=-0.018 -0.0899 -0.0759 rpy=0 0.349066 -1.5708
- joint LaserSensor/Shovel_sensor_fixedjoint: origin xyz=0.0562 0 -0.0692 rpy=0 0.349044 0 -> xyz=0.0562 0 -0.0692 rpy=0 0.349066 0
- joint LaserSensor/VerticalLeft_sensor_fixedjoint: origin xyz=0.0562 0 -0.0692 rpy=0 0.349044 0 -> xyz=0.0562 0 -0.0692 rpy=0 0.349066 0
- joint LaserSensor/VerticalRight_sensor_fixedjoint: origin xyz=0.0562 0 -0.0692 rpy=0 0.349044 0 -> xyz=0.0562 0 -0.0692 rpy=0 0.349066 0
- joint base_footprint_joint: child base_footprint -> Tibia; origin xyz=0 0 -0.334 rpy=0 0 0 -> xyz=0 0 0.334 rpy=0 0 0; parent Tibia -> base_footprint

Commit message: Update modifications, remove angular sign bug

File: share/urdf/pepper.urdf (robot description, URDF)
Before this commit: robot JulietteY20MP, 86 links, 85 joints
Links:
- removed link Lgrasp_frame
- link l_grasp_frame: mass 0 -> None
- link r_grasp_frame: mass 0 -> None
Joints:
- removed joint Lgrasp_frame_joint
- joint HipPitch: axis 0 1.0 0 -> 0 -1.0 0
- joint HipRoll: axis 1.0 0 0 -> -1.0 0 0
- joint KneePitch: axis 0 1.0 0 -> 0 -1.0 0
- joint LGrasp: axis 1.0 0 0 -> (none); limit lower=0.02 upper=0.98 effort=0.144 velocity=12.56 -> (none); origin xyz=0.05 0 0 rpy=-3.1415 0 1.5707 -> xyz=0.070 0 0 rpy=3.1415 0 1.5707
- joint RGrasp: axis 1.0 0 0 -> (none); limit lower=0.02 upper=0.98 effort=0.144 velocity=12.56 -> (none); origin xyz=0.05 0 0 rpy=-3.1415 0 1.5707 -> xyz=0.070 0 0 rpy=3.1415 0 1.5707

Commit message: Destroy torso base fixed frame, update intertia

File: share/urdf/pepper.urdf (robot description, URDF)
Before this commit: robot JulietteY20MP, 85 links, 84 joints
Links:
- removed link torso_base
Joints:
- removed joint torso_base_fixedjoint
- joint HipRoll: child torso_base -> torso; origin xyz=0 0 0.079 rpy=0 0 0 -> xyz=-2e-05 0 0.218 rpy=0 0 0

Commit message: Update urdf

File: share/urdf/pepper.urdf (robot description, URDF)
Before this commit: robot JulietteY20MP, 84 links, 83 joints
Links:
- removed link l_grasp_frame
- removed link r_grasp_frame
- link LFinger11_link: mass 2e-06 -> 2e-03
- link LFinger12_link: mass 2e-06 -> 2e-03
- link LFinger13_link: mass 2e-06 -> 2e-03
- link LFinger21_link: mass 2e-06 -> 2e-03
- link LFinger22_link: mass 2e-06 -> 2e-03
- link LFinger23_link: mass 2e-06 -> 2e-03
- link LFinger31_link: mass 2e-06 -> 2e-03
- link LFinger32_link: mass 2e-06 -> 2e-03
- link LFinger33_link: mass 2e-06 -> 2e-03
- link LFinger41_link: mass 2e-06 -> 2e-03
- link LFinger42_link: mass 2e-06 -> 2e-03
- link LFinger43_link: mass 2e-06 -> 2e-03
- link LThumb1_link: mass 2e-06 -> 2e-03
- link LThumb2_link: mass 2e-06 -> 2e-03
- link RFinger11_link: mass 2e-06 -> 2e-03
- link RFinger12_link: mass 2e-06 -> 2e-03
- link RFinger13_link: mass 2e-06 -> 2e-03
- link RFinger21_link: mass 2e-06 -> 2e-03
- link RFinger22_link: mass 2e-06 -> 2e-03
- link RFinger23_link: mass 2e-06 -> 2e-03
- link RFinger31_link: mass 2e-06 -> 2e-03
- link RFinger32_link: mass 2e-06 -> 2e-03
- link RFinger33_link: mass 2e-06 -> 2e-03
- link RFinger41_link: mass 2e-06 -> 2e-03
- link RFinger42_link: mass 2e-06 -> 2e-03
- link RFinger43_link: mass 2e-06 -> 2e-03
- link RThumb1_link: mass 2e-06 -> 2e-03
- link RThumb2_link: mass 2e-06 -> 2e-03
- link l_gripper: mass 2e-06 -> 2e-03
- link r_gripper: mass 2e-06 -> 2e-03
Joints:
- removed joint LGrasp
- removed joint RGrasp
- joint WheelFL: axis 1.0 0 0 -> 1.0 0.0 0.0
- joint WheelFR: axis 1.0 0 0 -> 1.0 0.0 0.0

Commit message: Update depth camera frame

File: share/urdf/pepper.urdf (robot description, URDF)
Before this commit: robot JulietteY20MP, 82 links, 81 joints
Joints:
- joint CameraDepth_sensor_fixedjoint: origin xyz=0.05138 0.039 0.1194 rpy=0 0 0 -> xyz=0.07618 0 0.1194 rpy=0 0 0

Commit message: Correct the hip roll link in the urdf

File: share/urdf/pepper.urdf (robot description, URDF)
Before this commit: robot JulietteY20MP, 82 links, 81 joints
Links:
- added link HipOffset, mass 0
Joints:
- added joint HipOffset_fixed: type fixed, parent HipOffset, child torso, origin xyz=0 0 0.139 rpy=0 0 0
- joint HipRoll: child torso -> HipOffset; origin xyz=-2e-05 0 0.218 rpy=0 0 0 -> xyz=-2e-05 0 0.079 rpy=0 0 0

Commit message: Correct URDF for the Hip Roll rotation

File: share/urdf/pepper.urdf (robot description, URDF)
Before this commit: robot JulietteY20MP, 83 links, 82 joints
Links:
- removed link HipOffset
Joints:
- removed joint HipOffset_fixed
- joint Accelerometer_sensor_fixedjoint: origin xyz=0.00239 -0.03575 0.00626 rpy=0 0 0 -> xyz=0.00239 -0.03575 0.14526 rpy=0 0 0
- joint ChestBoard/Button_sensor_fixedjoint: origin xyz=0.049871 0.001588 0.055163 rpy=0 0 0 -> xyz=0.049871 0.001588 0.194163 rpy=0 0 0
- joint Gyrometer_sensor_fixedjoint: origin xyz=0.00204 -0.03491 -0.00959 rpy=0 0 0 -> xyz=0.00204 -0.03491 0.12941 rpy=0 0 0
- joint HeadYaw: origin xyz=-0.038 0 0.1699 rpy=0 0 0 -> xyz=-0.038 0 0.3089 rpy=0 0 0
- joint HipRoll: child HipOffset -> torso
- joint LShoulderPitch: origin xyz=-0.057 0.14974 0.08682 rpy=0 0 0 -> xyz=-0.057 0.14974 0.22582 rpy=0 0 0
- joint RShoulderPitch: origin xyz=-0.057 -0.14974 0.08682 rpy=0 0 0 -> xyz=-0.057 -0.14974 0.22582 rpy=0 0 0
- joint Tablet_sensor_fixedjoint: origin xyz=0.0839249 0 0.06251 rpy=0 -0.523599 0 -> xyz=0.0839249 0 0.20151 rpy=0 -0.523599 0

Commit message: Revert depth camera frame position

File: share/urdf/pepper.urdf (robot description, URDF)
Before this commit: robot JulietteY20MP, 82 links, 81 joints
Joints:
- joint CameraDepth_sensor_fixedjoint: origin xyz=0.07618 0 0.1194 rpy=0 0 0 -> xyz=0.05138 0.039 0.1194 rpy=0 0 0

Commit message: Add base link to Pepper in order to have more consistency with NAO urdf

File: share/urdf/pepper.urdf (robot description, URDF)
Before this commit: robot JulietteY20MP, 82 links, 81 joints
Links:
- added link base_link
Joints:
- added joint base_link_joint: type fixed, parent base_link, child base_footprint, origin xyz=0 0 0 rpy=0 0 0

Commit message: Fixed r_gripper and l_gripper frames in the .urdf

File: share/urdf/pepper.urdf (robot description, URDF)
Before this commit: robot JulietteY20MP, 83 links, 82 joints
Links:
- added link l_hand, mass 2e-03
- added link r_hand, mass 2e-03
Joints:
- added joint LGripper: type fixed, parent l_wrist, child l_gripper, origin xyz=0.025 0 0 rpy=-2.355 0.0 -1.57, axis 0 0 0, limit lower=0.02 upper=0.98 effort=0.144 velocity=12.56
- added joint RGripper: type fixed, parent r_wrist, child r_gripper, origin xyz=0.025 0 0 rpy=2.355 0 1.57, axis 0 0 0, limit lower=0.02 upper=0.98 effort=0.144 velocity=12.56
- joint LHand: child l_gripper -> l_hand
- joint RHand: child r_gripper -> r_hand

Commit message: Change translation for the grasping frames

File: share/urdf/pepper.urdf (robot description, URDF)
Before this commit: robot JulietteY20MP, 85 links, 84 joints
Joints:
- joint LGripper: origin xyz=0.025 0 0 rpy=-2.355 0.0 -1.57 -> xyz=0.07 0.0 -0.01802319018 rpy=-2.355 0.0 -1.57
- joint RGripper: origin xyz=0.025 0 0 rpy=2.355 0 1.57 -> xyz=0.07 0.0 -0.01802319018 rpy=2.355 0 1.57

Commit message: Update the gripper frames

File: share/urdf/pepper.urdf (robot description, URDF)
Before this commit: robot JulietteY20MP, 85 links, 84 joints
Joints:
- joint LGripper: origin xyz=0.07 0.0 -0.01802319018 rpy=-2.355 0.0 -1.57 -> xyz=0.07 0.0 -0.01802319018 rpy=-3.14 0.0 -1.57
- joint RGripper: origin xyz=0.07 0.0 -0.01802319018 rpy=2.355 0 1.57 -> xyz=0.07 0.0 -0.01802319018 rpy=3.14 0 1.57

Commit message: Correct indent and remove unused lines

File: share/urdf/pepper.urdf (robot description, URDF)
Before this commit: robot JulietteY20MP, 85 links, 84 joints
Joints:
- joint LGripper: limit lower=0.02 upper=0.98 effort=0.144 velocity=12.56 -> (none)
- joint RGripper: limit lower=0.02 upper=0.98 effort=0.144 velocity=12.56 -> (none)
